Commit message: Updating Some Data

File: catkin_ws/src/robot_description_pkg/urdf/my_robot.xacro (robot description, xacro)
@@ -2,5 +2,12 @@
 <robot xmlns:xacro="http://www.ros.org/wiki/xacro" name="FourWheeledRobot">
     <xacro:include filename="$(find robot_description_pkg)/urdf/material.xacro" />
-    <xacro:include filename="$(find robot_description_pkg)/urdf/gazebo.gazebo" />
+    <xacro:include filename="$(find robot_description_pkg)/urdf/gazebo_plugins.gazebo" />
+    <!-- This is the footprint -->
+    <link name="robot_footprint"></link>
+    <joint name="robot_footprint_joint" type="fixed">
+        <origin xyz="0 0 0" rpy="0 0 0" />
+        <parent link="robot_footprint" />
+        <child link="chassis_link" />
+    </joint>
     <!-- This is the chassis -->
     <link name="chassis_link">

Commit message: intial commit

File: catkin_ws/src/robot_description_pkg/urdf/my_robot.xacro (robot description, xacro)
@@ -3,9 +3,9 @@
     <xacro:include filename="$(find robot_description_pkg)/urdf/material.xacro" />
     <xacro:include filename="$(find robot_description_pkg)/urdf/gazebo_plugins.gazebo" />
-    <!-- This is the footprint -->
-    <link name="robot_footprint"></link>
-    <joint name="robot_footprint_joint" type="fixed">
+    <!-- This is odom -->
+    <link name="odom"></link>
+    <joint name="odom_joint" type="fixed">
         <origin xyz="0 0 0" rpy="0 0 0" />
-        <parent link="robot_footprint" />
+        <parent link="odom" />
         <child link="chassis_link" />
     </joint>
@@ -24,5 +24,4 @@
             <material name="red">
                 <color rgba="1 0 0 1" />
-                <texture filename="" />
             </material>
         </visual>
@@ -34,4 +33,9 @@
         </collision>
     </link>
+    <gazebo reference="chassis_link">
+        <material name="red">
+            <color rgba="1 0 0 1" />
+        </material>
+    </gazebo>
     <!-- Back right wheel -->
     <joint name="wheel1_joint" type="continuous">
@@ -55,5 +59,4 @@
             <material name="yellow">
                 <color rgba="1 1 0 1" />
-                <texture filename="" />
             </material>
         </visual>
@@ -65,4 +68,9 @@
         </collision>
     </link>
+    <gazebo reference="wheel1_link">
+        <material name="yellow">
+            <color rgba="1 1 0 1" />
+        </material>
+    </gazebo>
     <!-- Back left wheel -->
     <joint name="wheel2_joint" type="continuous">
@@ -96,4 +104,9 @@
         </collision>
     </link>
+    <gazebo reference="wheel2_link">
+        <material name="yellow">
+            <color rgba="1 1 0 1" />
+        </material>
+    </gazebo>
     <!-- front right wheel -->
     <joint name="wheel3_joint" type="continuous">
@@ -127,4 +140,9 @@
         </collision>
     </link>
+    <gazebo reference="wheel3_link">
+        <material name="yellow">
+            <color rgba="1 1 0 1" />
+        </material>
+    </gazebo>
     <!-- front left wheel -->
     <joint name="wheel4_joint" type="continuous">
@@ -158,4 +176,9 @@
         </collision>
     </link>
+    <gazebo reference="wheel4_link">
+        <material name="yellow">
+            <color rgba="1 1 0 1" />
+        </material>
+    </gazebo>
     <!-- Camera -->
     <joint name="camera_joint" type="fixed">
